Commit message: mainly works

File: exprob_assignment3/urdf/robot31.urdf (robot description, URDF)
Before this commit: robot myrobot3, 12 links, 11 joints
Links:
- link left_grip_link: geometry collision box size=0 0 0; visual box size=0.001 0.001 0.001
- link right_grip_link: geometry collision box size=0 0 0; visual box size=0.001 0.001 0.001
